Commit message: Add base_link and add directories to share/

File: ros2_ws/src/arm_assembly_description/urdf/arm_assembly.xacro (robot description, xacro)
@@ -5,4 +5,7 @@
 <xacro:include filename="$(find arm_assembly_description)/urdf/arm_assembly.trans" />
 <xacro:include filename="$(find arm_assembly_description)/urdf/arm_assembly.gazebo" />
+  <!-- Base Link -->
+  <link name="base_link">
+  </link>
   <!-- Link dcmotor -->
   <link name="dcmotor">
@@ -317,4 +320,10 @@
     </collision>
   </link>
+  <!-- Joint from base_link to dcmotor -->
+  <joint name="dcmotor_to_base" type="fixed">
+    <parent link="base_link"/>
+    <child link="dcmotor"/>
+    <origin xyz="0.0 0.0 0.0" rpy="0.0 0.0 0.0"/>
+  </joint>
   <!-- Joint from motor_bracket to camera_support -->
   <joint name="camera_pitch" type="revolute">

Commit message: Make URDF Gazebo Compatible and add Launch Files

File: ros2_ws/src/arm_assembly_description/urdf/arm_assembly.xacro (robot description, xacro)
@@ -5,5 +5,8 @@
 <xacro:include filename="$(find arm_assembly_description)/urdf/arm_assembly.trans" />
 <xacro:include filename="$(find arm_assembly_description)/urdf/arm_assembly.gazebo" />
-  <!-- Base Link -->
+<!-- Link world -->
+<link name="world">
+</link>
+  <!-- Link Base -->
   <link name="base_link">
   </link>
@@ -320,10 +323,4 @@
     </collision>
   </link>
-  <!-- Joint from base_link to dcmotor -->
-  <joint name="dcmotor_to_base" type="fixed">
-    <parent link="base_link"/>
-    <child link="dcmotor"/>
-    <origin xyz="0.0 0.0 0.0" rpy="0.0 0.0 0.0"/>
-  </joint>
   <!-- Joint from motor_bracket to camera_support -->
   <joint name="camera_pitch" type="revolute">
@@ -358,3 +355,15 @@
     <limit effort="10" velocity="10" lower="-0.785398" upper="0.785398"/>
   </joint>
+  <!-- Joint from base_link to dcmotor -->
+  <joint name="dcmotor_to_base" type="fixed">
+    <parent link="base_link"/>
+    <child link="dcmotor"/>
+    <origin xyz="0.0 0.0 0.0" rpy="0.0 0.0 0.0"/>
+  </joint>
+  <!-- Joint from world to base_link -->
+  <joint name="world_to_base" type="fixed">
+    <child link="base_link"/>
+    <parent link="world"/>
+    <origin xyz="0.0 0.0 0.0" rpy="0.0 0.0 0.0"/>
+  </joint>
 </robot>

Commit message: Remove base_link and world joint

File: ros2_ws/src/arm_assembly_description/urdf/arm_assembly.xacro (robot description, xacro)
@@ -362,5 +362,5 @@
   </joint>
   <!-- Joint from world to base_link -->
-  <joint name="world_to_base" type="fixed">
+  <joint name="base_to_world" type="fixed">
     <child link="base_link"/>
     <parent link="world"/>
